File: hardware/0.1/avrisp-mkII.sch (KiCad schematic (older format))
At the start: 5 parts

Commit message: layout done
Parts:
- removed LOGO5: 4-Layer-Check, josh-logos:4-layer-check, symbol Mechanical:MountingHole
- added C1, C2, C7: 1u, Capacitor_SMD:C_0603_1608Metric, symbol Device:C
- added C10, C12, C3, C8, C9: 100n, Capacitor_SMD:C_0603_1608Metric, symbol Device:C
- added C11: 10u, Capacitor_SMD:C_0603_1608Metric, symbol Device:C
- added C4: 100u, Capacitor_Tantalum_SMD:CP_EIA-3216-10_Kemet-I, symbol Device:CP1
- added C5, C6: 22P, Capacitor_SMD:C_0603_1608Metric, symbol Device:C
- added D1: 1N4148, Diode_SMD:D_SOD-323, symbol Device:D
- added D2: PWR, LED_SMD:LED_0603_1608Metric, symbol Device:LED
- added D3: STAT, LED_SMD:LED_0603_1608Metric, symbol Device:LED
- added D4, D6: BAT54C, Package_TO_SOT_SMD:SOT-23, symbol Diode:BAT54C
- added D5: ACT, LED_SMD:LED_0603_1608Metric, symbol Device:LED
- added F1: 100mA, josh-passives-smt:Fuse_0805_2012Metric, symbol Device:Polyfuse_Small
- added FB1, FB2: 600R, josh-passives-smt:Ferrite_Bead_0603, symbol josh-passive:Ferrite_Bead_PWR
- added J1: USB_C_Receptacle_USB2.0, josh-connectors:USB_C_U262-161N-4BVC11, symbol Connector:USB_C_Receptacle_USB2.0
- added J2, J3: 2.54 THT, Connector_PinHeader_2.54mm:PinHeader_1x03_P2.54mm_Vertical, symbol Connector_Generic:Conn_01x03
- added J4: AVR ISP, Connector_IDC:IDC-Header_2x03_P2.54mm_Vertical, symbol Connector_Generic:Conn_02x03_Odd_Even
- added JP1: VCC_SEL, Jumper:SolderJumper-3_P1.3mm_Bridged12_Pad1.0x1.5mm, symbol Jumper:Jumper_3_Bridged12
- added R1, R2: 5K1, Resistor_SMD:R_0603_1608Metric, symbol Device:R
- added R3: 10K, Resistor_SMD:R_0603_1608Metric, symbol Device:R
- added R4: 100R, Resistor_SMD:R_0603_1608Metric, symbol Device:R
- added R5, R6: 22R, Resistor_SMD:R_0603_1608Metric, symbol Device:R
- added R8: 1M, Resistor_SMD:R_0603_1608Metric, symbol Device:R
- added R9: 200R, Resistor_SMD:R_0603_1608Metric, symbol Device:R
- added RN1, RN2: 1K, Resistor_SMD:R_Array_Convex_4x0603, symbol josh-passive:RN
- added SW1: RST, josh-buttons-switches:Panasonic_EVQPUL_EVQPUC, symbol Switch:SW_Push
- added SW2: SW_Push, josh-buttons-switches:Panasonic_EVQPUL_EVQPUC, symbol Switch:SW_Push
- added U1: USBLC6-2SC6, Package_TO_SOT_SMD:SOT-23-6, symbol josh-ic:USBLC6-2SC6
- added U2: AP2112K-3.3, Package_TO_SOT_SMD:SOT-23-5, symbol Regulator_Linear:AP2112K-3.3
- added U3: MCP130-xxxxTT, Package_TO_SOT_SMD:SOT-23, symbol Power_Supervisor:MCP130-xxxxTT
- added U4: AT90USB162-16AU, Package_QFP:TQFP-32_7x7mm_P0.8mm, symbol MCU_Microchip_AVR:AT90USB162-16AU
- added Y1: 16MHz, josh-oscillators:Crystal_SMD_3225-4Pin_3.2x2.5mm, symbol Device:Crystal_GND24_Small
- renumbered LOGO3 to LOGO1, LOGO4 to LOGO2, LOGO1 to LOGO3, LOGO2 to LOGO4
Connections:
- net labels added: +5V, D+, D-, GND, ICSP_MISO, ICSP_MOSI, ICSP_RST, ICSP_SCK, LED_ACTIVITY, LED_READY, LED_USB_PWR, PB1(SCK), PB2(MOSI), PB3(MISO), PB4(TARG_RST), RST, USB_D+, USB_D-, USB_PWR_DET, VCC, V_TARGET
- wire segments 0 -> 214
- no-connect marks 0 -> 14
Other:
- note added: "MCU VOLATAGE \nSELECTON"
- note added: "TARGET VOLTAGE SEL"
- note added: "USB PWR ON / OFF"
- note added: "Voltage Supervisor"
